File: Antennas files/Antennas_PCB/Antennas_PCB.kicad_pcb (KiCad board)
At the start: 2 copper layers, 11 parts, among them U1 LMR14030SDDA, U2 TSR_1-2433

Commit message: Add files via upload
pcb design for new buck and volt reg
Parts:
- removed CBOOT1: 0.1uF, Capacitor_SMD:C_0805_2012Metric_Pad1.18x1.45mm_HandSolder
- removed COUT2: 10uF, Capacitor_SMD:C_1206_3216Metric_Pad1.33x1.80mm_HandSolder
- removed CSS1: 22nF, Capacitor_SMD:C_0805_2012Metric_Pad1.18x1.45mm_HandSolder
- removed RT1: 49.9kO, Resistor_SMD:R_0805_2012Metric_Pad1.20x1.40mm_HandSolder
- removed U1: LMR14030SDDA, Package_SO:Texas_R-PDSO-G8_EP2.95x4.9mm_Mask2.4x3.1mm
- added BUCK: LM2576T-ADJ, Package_TO_SOT_THT:TO-220-5_Vertical, F.Cu at (121.1, 46.9)
- added CIN3: 100uF, Capacitor_THT:C_Disc_D5.0mm_W2.5mm_P5.00mm, F.Cu at (116.2, 46.8)
- added D1: 1N5822, Diode_THT:D_DO-201AD_P12.70mm_Horizontal, F.Cu at (122.5, 58.7)
- added J1: Conn_01x02_Pin, Connector_PinHeader_1.00mm:PinHeader_1x02_P1.00mm_Vertical, F.Cu at (106.0, 49.5)
- added J2: Conn_01x02_Pin, Connector_PinHeader_1.00mm:PinHeader_1x02_P1.00mm_Vertical, F.Cu at (151.9, 50.5)
- added L1: 100uH, Inductor_THT:L_Axial_L6.6mm_D2.7mm_P10.16mm_Horizontal_Vishay_IM-2, F.Cu at (122.6, 52.4)
- added PMOS: PMOS, my_library:Untitled, F.Cu at (112.6, 49.4)
- CIN1: value 4.7uF -> 1000uF; footprint Capacitor_SMD:C_0805_2012Metric_Pad1.18x1.45mm_HandSolder -> Capacitor_THT:C_Disc_D5.0mm_W2.5mm_P5.00mm
- CIN2: footprint Capacitor_SMD:C_0805_2012Metric_Pad1.18x1.45mm_HandSolder -> Capacitor_THT:C_Disc_D5.0mm_W2.5mm_P5.00mm
- COUT1: footprint Capacitor_SMD:C_1206_3216Metric_Pad1.33x1.80mm_HandSolder -> Capacitor_THT:C_Disc_D5.0mm_W2.5mm_P5.00mm
- R1: value 17.8kO -> 20kO; footprint Resistor_SMD:R_0805_2012Metric_Pad1.20x1.40mm_HandSolder -> Resistor_THT:R_Axial_DIN0207_L6.3mm_D2.5mm_P10.16mm_Horizontal
- R2: value 100k -> 62kO; footprint Resistor_SMD:R_0805_2012Metric_Pad1.20x1.40mm_HandSolder -> Resistor_THT:R_Axial_DIN0207_L6.3mm_D2.5mm_P10.16mm_Horizontal
- U2: value TSR_1-2433 -> LD1117V33; footprint Converter_DCDC:Converter_DCDC_TRACO_TSR-1_THT -> Package_TO_SOT_THT:TO-220-3_Vertical
- moved R1 36.2 mm to (121.6, 41.1), turned to 180 degrees
- moved U2 35.6 mm to (141.6, 50.9), turned to 90 degrees
- moved R2 32.3 mm to (136.3, 41.1), turned to 180 degrees
- moved CIN2 31.6 mm to (135.8, 44.2), turned to -90 degrees
- moved COUT1 30.2 mm to (146.7, 48.5), turned to -90 degrees
- moved CIN1 24.4 mm to (132.1, 49.2), turned to 90 degrees
Connections:
- CIN1 pad 1: +24V -> /V_OUT_BUCK(5V)
- CIN2 pad 1: +24V -> /V_OUT_BUCK(5V)
- COUT1 pad 1: /V_BUCK_OUT -> /V_OUT(3.3V)
- R2 pad 1: /V_BUCK_OUT -> /V_OUT_BUCK(5V)
- U2 pad 1: /V_BUCK_OUT -> GND
- U2 pad 2: GND -> /V_OUT(3.3V)
- U2 pad 3: /ESP_VIN -> /V_OUT_BUCK(5V)
Routing:
- net /V_OUT_BUCK(5V): track 0.00 -> 20.0 mm
- net /OUT: track 0.00 -> 12.1 mm
- net /V_OUT(3.3V): track 0.00 -> 10.8 mm
- net /FB: track 0.00 -> 10.3 mm
- net /VIN: track 0.00 -> 10.1 mm
- net Net-(J1-Pin_1): track 0.00 -> 5.12 mm
- added copper zone on F.Cu, net GND
Other:
- board text added: "Antenna pcb for suplying"
- board text added: "GND"
- board text added: "VIN"
- board text added: "VS"
