File: PCB/SPRO-3.kicad_pcb (KiCad board)
At the start: 2 copper layers, 46 parts, among them J1 Screw_Terminal_01x02, J2 Micro_SD_Card, Q1 IRF4905, U1 TSR_1-2450, U2 ESP32-S3-DEVKITC-1-N8R2, U6 LD1117V33

Commit message: Add files via upload
Parts:
- moved R14 131.7 mm to (113.1, 126.5), turned to 180 degrees
- moved R12 126.0 mm to (113.2, 111.2), turned to 180 degrees
- moved R15 122.4 mm to (102.5, 126.2), turned to -90 degrees
- moved R10 120.5 mm to (113.2, 96.2), turned to 180 degrees
- moved R13 116.5 mm to (102.8, 111.0), turned to -90 degrees
- moved R18 111.8 mm to (150.5, 30.3), turned to 180 degrees
- moved R11 110.7 mm to (102.8, 95.9), turned to -90 degrees
- moved R24 104.8 mm to (150.2, 46.8), turned to 180 degrees
- moved J_US3 100.5 mm to (116.0, 121.2)
- moved R17 100.4 mm to (139.1, 30.3), turned to 180 degrees
- moved R4 99.1 mm to (23.7, 112.8)
- moved R5 99.1 mm to (23.7, 116.8)
- moved R6 99.1 mm to (23.7, 120.8)
- moved J_MD1 98.5 mm to (124.0, 30.5)
- moved R23 92.8 mm to (138.9, 46.8), turned to 180 degrees
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- renumbered R20 to R19, R19 to R20, R24 to R23, R23 to R24

Commit message: Add files via upload
Parts:
- added J3: Conn_01x22, Connector_PinHeader_2.54mm:PinHeader_1x22_P2.54mm_Vertical, F.Cu at (118.4, 51.8)
- added J4: Conn_01x22, Connector_PinHeader_2.54mm:PinHeader_1x22_P2.54mm_Vertical, F.Cu at (152.9, 51.8)
- added J_Motor1: Screw_Terminal_01x02, TerminalBlock_Phoenix:TerminalBlock_Phoenix_MKDS-1,5-2-5.08_1x02_P5.08mm_Horizontal, F.Cu at (60.9, 24.3)
- added J_Motor2: Screw_Terminal_01x02, TerminalBlock_Phoenix:TerminalBlock_Phoenix_MKDS-1,5-2-5.08_1x02_P5.08mm_Horizontal, F.Cu at (72.8, 24.2)
- added J_Switch1: Screw_Terminal_01x02, TerminalBlock_Phoenix:TerminalBlock_Phoenix_MKDS-1,5-2-5.08_1x02_P5.08mm_Horizontal, F.Cu at (24.9, 25.9)
- J1: footprint Connector_PinHeader_2.54mm:PinHeader_1x02_P2.54mm_Vertical -> TerminalBlock_Phoenix:TerminalBlock_Phoenix_MKDS-1,5-2-5.08_1x02_P5.08mm_Horizontal
- moved J_US1 94.2 mm to (26.2, 63.6)
- moved J_US2 94.1 mm to (26.2, 78.8)
- moved C5 93.9 mm to (110.6, 90.9), turned to -90 degrees
- moved J_US3 93.9 mm to (26.2, 93.8)
- moved R12 84.3 mm to (33.5, 84.0), turned to -90 degrees
- moved R10 84.3 mm to (33.5, 69.0), turned to -90 degrees
- moved R14 83.8 mm to (33.5, 100.0), turned to -90 degrees
- moved U2 65.2 mm to (135.7, 81.7)
- moved R11 65.2 mm to (40.5, 76.7), turned to 90 degrees
- moved R13 65.1 mm to (40.5, 91.7), turned to 90 degrees
- moved R15 64.7 mm to (40.5, 107.7), turned to 90 degrees
- moved J2 64.4 mm to (98.8, 81.9), turned to 180 degrees
- moved R1 61.4 mm to (110.2, 78.4), turned to -90 degrees
- moved R6 50.4 mm to (72.1, 106.7), turned to 90 degrees
- moved R24 49.7 mm to (100.5, 45.8), turned to -90 degrees
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Connections:
- Q1 pad 3: Net-(J1-Pin_1) -> Net-(J_Switch1-Pin_1)
- U2 pad J1_14: unconnected-(U2-GPIO46-PadJ1_14) -> GPIO46
- U2 pad J1_3: unconnected-(U2-RST-PadJ1_3) -> RST
- U2 pad J3_10: unconnected-(U2-GPIO38-PadJ3_10) -> GPIO38
- U2 pad J3_11: unconnected-(U2-GPIO37-PadJ3_11) -> GPIO37
- U2 pad J3_12: unconnected-(U2-GPIO36-PadJ3_12) -> GPIO36
- U2 pad J3_13: unconnected-(U2-GPIO35-PadJ3_13) -> GPIO35
- U2 pad J3_14: unconnected-(U2-GPIO0-PadJ3_14) -> GPIO0
- U2 pad J3_16: unconnected-(U2-GPIO48-PadJ3_16) -> GPIO48
- U2 pad J3_17: unconnected-(U2-GPIO47-PadJ3_17) -> GPIO47
- U2 pad J3_2: unconnected-(U2-U0TXD/GPIO43-PadJ3_2) -> U0TXD/GPIO43
- U2 pad J3_3: unconnected-(U2-U0RXD/GPIO44-PadJ3_3) -> U0RXD/GPIO44
- U2 pad J3_7: unconnected-(U2-MTDI/GPIO41-PadJ3_7) -> GPIO41
- U2 pad J3_8: unconnected-(U2-MTDO/GPIO40-PadJ3_8) -> GPIO40
- U2 pad J3_9: unconnected-(U2-MTCK/GPIO39-PadJ3_9) -> GPIO39
Routing:
- net +5V: track 0.00 -> 364.3 mm
- net +3.3V: track 0.00 -> 247.4 mm, vias 0 -> 1
- net +12V: track 0.00 -> 177.5 mm, vias 0 -> 38
- net GPIO18: track 0.00 -> 151.2 mm
- net GPIO42: track 0.00 -> 130.3 mm, vias 0 -> 2
- net GPIO19: track 0.00 -> 130.0 mm, vias 0 -> 1
- net GPIO20: track 0.00 -> 127.0 mm, vias 0 -> 1
- net GPIO21: track 0.00 -> 115.4 mm, vias 0 -> 1
- net GPIO14: track 0.00 -> 112.2 mm
- net GPIO16: track 0.00 -> 105.6 mm, vias 0 -> 2
- net GPIO1: track 0.00 -> 104.8 mm
- net GPIO17: track 0.00 -> 102.3 mm, vias 0 -> 3
- net GPIO15: track 0.00 -> 100.4 mm, vias 0 -> 2
- net GPIO2: track 0.00 -> 93.5 mm
- net GPIO45: track 0.00 -> 78.3 mm
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- added copper zone on B.Cu, net GND
Other:
- board outline added: 140.1 x 102.4 mm

Commit message: Add files via upload
Parts:
- added R25: 47kΩ, Resistor_THT:R_Axial_DIN0207_L6.3mm_D2.5mm_P7.62mm_Horizontal, F.Cu at (85.6, 93.9)
- added R26: 47kΩ, Resistor_THT:R_Axial_DIN0207_L6.3mm_D2.5mm_P7.62mm_Horizontal, F.Cu at (107.9, 96.2)
- R11, R13, R15: value 2kΩ -> 1.8kΩ
Connections:
- J2 pad 1: unconnected-(J2-DAT2-Pad1) -> Net-(J2-DAT2)
- J2 pad 8: unconnected-(J2-DAT1-Pad8) -> Net-(J2-DAT1)
Routing:
- net +3.3V: track 247.4 -> 275.1 mm
- net Net-(J2-DAT2): track 0.00 -> 12.4 mm, vias 0 -> 3
- net Net-(J2-DAT1): track 0.00 -> 9.24 mm, vias 0 -> 2
- net GPIO 13 / MISO: track 54.6 -> 57.1 mm
- net +5V: track 364.3 -> 366.3 mm
- net GND: track 58.1 -> 60.0 mm, vias 6 -> 7
- net GPIO 11 / MOSI: track 49.8 -> 51.1 mm
- net GPIO 12 / SCK: track 31.3 -> 32.3 mm
Other:
- board text added: "GND"
- board text added: "VCC"

Commit message: Add files via upload
Parts:
- added J_Encoder_1: Conn_01x04, Connector_PinHeader_2.54mm:PinHeader_1x04_P2.54mm_Vertical, F.Cu at (119.4, 21.2)
- added J_Encoder_2: Conn_01x04, Connector_PinHeader_2.54mm:PinHeader_1x04_P2.54mm_Vertical, F.Cu at (141.6, 21.1)
- added R27: 1kΩ, Resistor_THT:R_Axial_DIN0207_L6.3mm_D2.5mm_P7.62mm_Horizontal, F.Cu at (114.5, 29.7)
- added R28: 1.8kΩ, Resistor_THT:R_Axial_DIN0207_L6.3mm_D2.5mm_P7.62mm_Horizontal, F.Cu at (109.8, 22.1)
- added R29: 1kΩ, Resistor_THT:R_Axial_DIN0207_L6.3mm_D2.5mm_P7.62mm_Horizontal, F.Cu at (124.1, 29.7)
- added R30: 1.8kΩ, Resistor_THT:R_Axial_DIN0207_L6.3mm_D2.5mm_P7.62mm_Horizontal, F.Cu at (128.2, 29.7)
- added R31: 1kΩ, Resistor_THT:R_Axial_DIN0207_L6.3mm_D2.5mm_P7.62mm_Horizontal, F.Cu at (136.8, 29.5)
- added R32: 1.8kΩ, Resistor_THT:R_Axial_DIN0207_L6.3mm_D2.5mm_P7.62mm_Horizontal, F.Cu at (133.3, 21.8)
- added R33: 1kΩ, Resistor_THT:R_Axial_DIN0207_L6.3mm_D2.5mm_P7.62mm_Horizontal, F.Cu at (146.0, 29.4)
- added R34: 1.8kΩ, Resistor_THT:R_Axial_DIN0207_L6.3mm_D2.5mm_P7.62mm_Horizontal, F.Cu at (150.0, 29.4)
- moved R21 5.48 mm to (86.7, 48.9)
- moved J_MD1 5.48 mm to (91.3, 21.3)
- moved R18 5.48 mm to (104.1, 23.9)
- moved R19 5.48 mm to (86.4, 31.4)
- moved R20 5.48 mm to (81.3, 23.8)
- moved R17 5.48 mm to (98.9, 31.5)
- moved R22 5.48 mm to (81.5, 41.2)
- moved J_MD2 5.48 mm to (91.3, 36.9)
- moved R23 5.48 mm to (98.7, 48.9)
- moved R24 5.48 mm to (103.7, 41.3)
Connections:
- J_HX711_LC1 pad 4: GPIO45 -> GPIO35
Routing:
- net GPIO35: track 5.84 -> 84.1 mm
- net GPIO36: track 5.84 -> 79.1 mm, vias 0 -> 2
- net GPIO45: track 78.3 -> 5.84 mm
- net GPIO37: track 5.84 -> 73.1 mm, vias 0 -> 2
- net GPIO38: track 5.84 -> 66.2 mm, vias 0 -> 2
- net GPIO39: track 5.84 -> 55.2 mm, vias 0 -> 1
- net +5V: track 366.3 -> 400.8 mm
- net GND: track 60.0 -> 76.0 mm, vias 7 -> 8
- net Net-(J_Encoder_2-Pin_4): track 0.00 -> 8.70 mm
- net Net-(J_Encoder_1-Pin_4): track 0.00 -> 8.68 mm
- net Net-(J_Encoder_1-Pin_3): track 0.00 -> 7.41 mm
- net Net-(J_Encoder_2-Pin_3): track 0.00 -> 6.48 mm
- net GPIO1: track 104.8 -> 100.5 mm
- net GPIO6: track 51.4 -> 55.1 mm
- net GPIO2: track 93.5 -> 89.7 mm
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Other:
- outline, holes or cut-outs redrawn
- board text added: "CLK"
- board text added: "DAT"
- board text added: "R L"
- board text added: "VDD"

Commit message: final pcb
Parts:
- removed R17, R19, R21, R23: 1.8kΩ, Resistor_THT:R_Axial_DIN0207_L6.3mm_D2.5mm_P7.62mm_Horizontal
- R18, R20, R22, R24: value 3.3kΩ -> 3.9kΩ
- moved R18 5.20 mm to (98.9, 23.9)
- moved R20 5.20 mm to (86.5, 23.8)
- moved R22 5.00 mm to (86.5, 41.2)
- moved R24 5.00 mm to (98.7, 41.3)
Connections:
- J_MD1 pad 3: Net-(J_MD1-Pin_4) -> GPIO1
- J_MD1 pad 4: Net-(J_MD1-Pin_3) -> GPIO2
- J_MD2 pad 3: Net-(J_MD2-Pin_4) -> GPIO3
- J_MD2 pad 4: Net-(J_MD2-Pin_3) -> GPIO4
Routing:
- net GPIO2: track 89.7 -> 99.5 mm
- net GPIO4: track 32.7 -> 41.4 mm
- net GPIO3: track 57.6 -> 63.9 mm
- net Net-(J_MD2-Pin_3): track 5.57 -> 0.00 mm
- net Net-(J_MD2-Pin_4): track 5.43 -> 0.00 mm
- net Net-(J_MD1-Pin_3): track 5.12 -> 0.00 mm
- net Net-(J_MD1-Pin_4): track 4.94 -> 0.00 mm
- net GPIO1: track 100.5 -> 104.9 mm
