File: PCB/SPRO-3.kicad_sch (KiCad schematic)
At the start: 48 parts, among them J1 Screw_Terminal_01x02, J2 Micro_SD_Card, Q1 IRF4905, U2 ESP32-S3-DEVKITC-1-N8R2, U5 LM2576T-ADJ, U6 LD1117V33

Commit message: finalized the schematic
Parts:
- removed D1: 1N5822, Diode_THT:D_DO-201AD_P15.24mm_Horizontal, symbol Diode:1N5822
- removed L1: 100µH, symbol Device:L
- removed U5: LM2576T-ADJ, Package_TO_SOT_THT:TO-220-5_Vertical, symbol Regulator_Switching:LM2576T-ADJ
- added U1: TSR_1-2450, Converter_DCDC:Converter_DCDC_TRACO_TSR-1_THT, symbol Converter_DCDC:TSR_1-2450
- C1: value 100µF -> 10µF; footprint (none) -> Capacitor_THT:CP_Radial_D5.0mm_P2.00mm
- C2: value 1000µF -> 10µF; footprint (none) -> Capacitor_THT:CP_Radial_D5.0mm_P2.00mm
- C3, C7: footprint (none) -> Capacitor_THT:C_Disc_D5.0mm_W2.5mm_P2.50mm
- C4, C5: footprint (none) -> Capacitor_THT:CP_Radial_D5.0mm_P2.00mm
- C6: footprint (none) -> Capacitor_THT:CP_Radial_D6.3mm_P2.50mm
- J1: footprint (none) -> Connector_PinHeader_2.54mm:PinHeader_1x02_P2.54mm_Vertical
- J_HX711_LC1: renamed from J_HX711_LC; footprint (none) -> Connector_PinHeader_2.54mm:PinHeader_1x05_P2.54mm_Vertical
- J_IR1: renamed from J_IR; footprint (none) -> Connector_PinHeader_2.54mm:PinHeader_2x02_P2.54mm_Vertical
- J_IR2, J_IR3: footprint (none) -> Connector_PinHeader_2.54mm:PinHeader_2x02_P2.54mm_Vertical
- J_MD1, J_MD2: footprint (none) -> Connector_PinHeader_2.54mm:PinHeader_2x04_P2.54mm_Vertical
- J_US1, J_US2, J_US3: footprint (none) -> Connector_PinHeader_2.54mm:PinHeader_1x04_P2.54mm_Vertical
- R1, R10, R11, R12, R13, R14, R15, R16, R17, R18, R19, R2, R20, R21, R22, R23, R24, R3, R4, R5, R6, R7, R8, R9: footprint (none) -> Resistor_THT:R_Axial_DIN0207_L6.3mm_D2.5mm_P7.62mm_Horizontal
Connections:
- net +12V: now also U1.1 (Vin)
- net +3.3V: now also J_HX711_LC1.1 (Pin_1); no longer J_HX711_LC1.VDD (Pin_1)
- net +5V: now also J_HX711_LC1.2 (Pin_2), J_MD1.1 (Pin_2), J_MD1.5 (Pin_6), J_MD1.6 (Pin_5), J_MD2.1 (Pin_2), J_MD2.5 (Pin_6), J_MD2.6 (Pin_5), J_US1.1 (Pin_1), J_US2.1 (Pin_1), J_US3.1 (Pin_1), U1.3 (Vout); no longer J_HX711_LC1.VCC (Pin_2), J_MD1.L_EN (Pin_5), J_MD1.R_EN (Pin_6), J_MD1.VCC (Pin_2), J_MD2.L_EN (Pin_5), J_MD2.R_EN (Pin_6), J_MD2.VCC (Pin_2), J_US1.VCC (Pin_1), J_US2.VCC (Pin_1), J_US3.VCC (Pin_1)
- net GND: now also J2.10 (CD2), J2.9 (CD1), J_HX711_LC1.5 (Pin_5), J_MD1.2 (Pin_1), J_MD2.2 (Pin_1), J_US1.4 (Pin_4), J_US2.4 (Pin_4), J_US3.4 (Pin_4), U1.2 (GND); no longer J_HX711_LC1.GND (Pin_5), J_MD1.GND (Pin_1), J_MD2.GND (Pin_1), J_US1.GND (Pin_4), J_US2.GND (Pin_4), J_US3.GND (Pin_4)
- net GPIO14: now also J_US1.2 (Pin_2); no longer J_US1.Trig (Pin_2)
- net GPIO16: now also J_US2.2 (Pin_2); no longer J_US2.Trig (Pin_2)
- net GPIO18: now also J_US3.2 (Pin_2); no longer J_US3.Trig (Pin_2)
- net GPIO45: now also J_HX711_LC1.4 (Pin_4); no longer J_HX711_LC1.CLK (Pin_4)
- net GPIO5: now also J_MD1.7 (Pin_8); no longer J_MD1.RPWM (Pin_8)
- net GPIO6: now also J_MD1.8 (Pin_7); no longer J_MD1.LPWM (Pin_7)
- net GPIO7: now also J_MD2.7 (Pin_8); no longer J_MD2.RPWM (Pin_8)
- net GPIO8: now also J_MD2.8 (Pin_7); no longer J_MD2.LPWM (Pin_7)
- net GPIO9: now also J_HX711_LC1.3 (Pin_3); no longer J_HX711_LC1.DAT (Pin_3)
- net at R24.2: now also J_MD2.4 (Pin_3); no longer J_MD2.L_IS (Pin_3)
- net at R14.1: now also J_US3.3 (Pin_3); no longer J_US3.Echo (Pin_3)
- net at R12.1: now also J_US2.3 (Pin_3); no longer J_US2.Echo (Pin_3)
- net at R17.2: now also J_MD1.4 (Pin_3); no longer J_MD1.L_IS (Pin_3)
- net at R20.2: now also J_MD1.3 (Pin_4); no longer J_MD1.R_IS (Pin_4)
- net at R21.2: now also J_MD2.3 (Pin_4); no longer J_MD2.R_IS (Pin_4)
- net at R10.1: now also J_US1.3 (Pin_3); no longer J_US1.Echo (Pin_3)
Other:
- moved on the sheet: C3, C4, C5, R1, R10, R11, R12, R13, R14, R15, R17, R18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

Commit message: Add files via upload
Parts:
- added J3, J4: Conn_01x22, Connector_PinHeader_2.54mm:PinHeader_1x22_P2.54mm_Vertical, symbol Connector_Generic:Conn_01x22
- added J_Switch1: Conn_01x03, Connector_PinHeader_2.54mm:PinHeader_1x03_P2.54mm_Vertical, symbol Connector_Generic:Conn_01x03
- renumbered R20 to R19, R19 to R20, R24 to R23, R23 to R24
Connections:
- net +3.3V: now also J3.1 (Pin_1), J3.2 (Pin_2)
- net +5V: now also J3.21 (Pin_21)
- net GND: now also J3.22 (Pin_22), J4.1 (Pin_1), J4.21 (Pin_21), J4.22 (Pin_22)
- net GPIO 10 / CS: now also J3.16 (Pin_16)
- net GPIO 11 / MOSI: now also J3.17 (Pin_17)
- net GPIO 12 / SCK: now also J3.18 (Pin_18)
- net GPIO 13 / MISO: now also J3.19 (Pin_19)
- net GPIO1: now also J4.4 (Pin_4)
- net GPIO14: now also J3.20 (Pin_20)
- net GPIO15: now also J3.8 (Pin_8)
- net GPIO16: now also J3.9 (Pin_9)
- net GPIO17: now also J3.10 (Pin_10)
- net GPIO18: now also J3.11 (Pin_11)
- net GPIO19: no longer U2.J3_20 (USB_D-/GPIO19)
- net GPIO2: now also J4.5 (Pin_5)
- net GPIO20: no longer U2.J3_19 (USB_D+/GPIO20)
- net GPIO21: now also J4.18 (Pin_18)
- net GPIO3: now also J3.13 (Pin_13)
- net GPIO4: now also J3.4 (Pin_4)
- net GPIO42: no longer U2.J3_6 (MTMS/GPIO42)
- net GPIO45: now also J4.15 (Pin_15)
- net GPIO5: now also J3.5 (Pin_5)
- net GPIO6: now also J3.6 (Pin_6)
- net GPIO7: now also J3.7 (Pin_7)
- net GPIO8: now also J3.12 (Pin_12)
- net GPIO9: now also J3.15 (Pin_15)
- net at J1.1 (Pin_1): now also J_Switch1.2 (Pin_2); no longer Q1.3 (S)
- net GPIO46: now reaches U2.J1_14 (GPIO46)
- net GPIO46: now also J3.14 (Pin_14)
- net RST: now reaches U2.J1_3 (RST)
- net RST: now also J3.3 (Pin_3)
- net GPIO38: now reaches U2.J3_10 (GPIO38)
- net GPIO38: now also J4.10 (Pin_10)
- net GPIO37: now reaches U2.J3_11 (GPIO37)
- net GPIO37: now also J4.11 (Pin_11)
- net GPIO36: now reaches U2.J3_12 (GPIO36)
- net GPIO36: now also J4.12 (Pin_12)
- net GPIO35: now reaches U2.J3_13 (GPIO35)
- net GPIO35: now also J4.13 (Pin_13)
- net GPIO0: now reaches U2.J3_14 (GPIO0)
- net GPIO0: now also J4.14 (Pin_14)
- net GPIO48: now reaches U2.J3_16 (GPIO48)
- net GPIO48: now also J4.16 (Pin_16)
- net GPIO47: now reaches U2.J3_17 (GPIO47)
- net GPIO47: now also J4.17 (Pin_17)
- net U0TXD/GPIO43: now reaches U2.J3_2 (U0TXD/GPIO43)
- net U0TXD/GPIO43: now also J4.2 (Pin_2)
- net U0RXD/GPIO44: now reaches U2.J3_3 (U0RXD/GPIO44)
- net U0RXD/GPIO44: now also J4.3 (Pin_3)
- net MTDI/GPIO41: now reaches U2.J3_7 (MTDI/GPIO41)
- net MTDI/GPIO41: now also J4.7 (Pin_7)
- net MTDO/GPIO40: now reaches U2.J3_8 (MTDO/GPIO40)
- net MTDO/GPIO40: now also J4.8 (Pin_8)
- net MICK/GPIO39: now reaches U2.J3_9 (MTCK/GPIO39)
- net MICK/GPIO39: now also J4.9 (Pin_9)
- new net: J_Switch1.1 (Pin_1), Q1.3 (S)
- new net MTMS/GPIO42: J4.6 (Pin_6), U2.J3_6 (MTMS/GPIO42)
- new net USB_D+/GPIO20: J4.19 (Pin_19), U2.J3_19 (USB_D+/GPIO20)
- new net USB_D-/GPIO19: J4.20 (Pin_20), U2.J3_20 (USB_D-/GPIO19)
- no-connect marks 16 -> 3
Other:
- moved on the sheet: C6, C7, J1, J_HX711_LC1, Q1, R16, U2

Commit message: Add files via upload
Parts:
- removed J_Switch1: Conn_01x03, Connector_PinHeader_2.54mm:PinHeader_1x03_P2.54mm_Vertical, symbol Connector_Generic:Conn_01x03
- added J_Motor1, J_Motor2, J_Switch1: Screw_Terminal_01x02, TerminalBlock_Phoenix:TerminalBlock_Phoenix_MKDS-1,5-2-5.08_1x02_P5.08mm_Horizontal, symbol Connector:Screw_Terminal_01x02
- J1: footprint Connector_PinHeader_2.54mm:PinHeader_1x02_P2.54mm_Vertical -> TerminalBlock_Phoenix:TerminalBlock_Phoenix_MKDS-1,5-2-5.08_1x02_P5.08mm_Horizontal
Connections:
- net MTMS/GPIO42 is gone; now on net GPIO42: J4.6 (Pin_6), U2.J3_6 (MTMS/GPIO42)
- net USB_D+/GPIO20 is gone; now on net GPIO20: J4.19 (Pin_19), U2.J3_19 (USB_D+/GPIO20)
- net USB_D-/GPIO19 is gone; now on net GPIO19: J4.20 (Pin_20), U2.J3_20 (USB_D-/GPIO19)
- net +12V: now also J_Motor1.1 (Pin_1), J_Motor2.1 (Pin_1)
- net GND: now also J_Motor1.2 (Pin_2), J_Motor2.2 (Pin_2)
- net at J1.1 (Pin_1): now also J_Switch1.2 (Pin_2)
- net at Q1.3 (S): now also J_Switch1.1 (Pin_1)
- net MICK/GPIO39 renamed GPIO39
- net MTDI/GPIO41 renamed GPIO41
- net MTDO/GPIO40 renamed GPIO40
Other:
- moved on the sheet: C6, C7, Q1, R16

Commit message: Add files via upload
Parts:
- added R25, R26: 47kΩ, Resistor_THT:R_Axial_DIN0207_L6.3mm_D2.5mm_P7.62mm_Horizontal, symbol Device:R
- R11, R13, R15: value 2kΩ -> 1.8kΩ
Connections:
- net +3.3V: now also R25.1, R26.1
- net at J2.1 (DAT2): now also R26.2
- net at J2.8 (DAT1): now also R25.2
- no-connect marks 3 -> 1

Commit message: Add files via upload
Parts:
- added J_Encoder_1, J_Encoder_2: Conn_01x04, Connector_PinHeader_2.54mm:PinHeader_1x04_P2.54mm_Vertical, symbol Connector_Generic:Conn_01x04
- added R27, R29, R31, R33: 1kΩ, Resistor_THT:R_Axial_DIN0207_L6.3mm_D2.5mm_P7.62mm_Horizontal, symbol Device:R
- added R28, R30, R32, R34: 1.8kΩ, Resistor_THT:R_Axial_DIN0207_L6.3mm_D2.5mm_P7.62mm_Horizontal, symbol Device:R
Connections:
- net +5V: now also J_Encoder_1.2 (Pin_2), J_Encoder_2.2 (Pin_2)
- net GND: now also J_Encoder_1.1 (Pin_1), J_Encoder_2.1 (Pin_1), R28.1, R30.2, R32.1, R34.2
- net GPIO35: now also J_HX711_LC1.4 (Pin_4)
- net GPIO36: now also R27.1, R28.2
- net GPIO37: now also R29.1, R30.1
- net GPIO38: now also R31.1, R32.2
- net GPIO39: now also R33.1, R34.1
- net GPIO45: no longer J_HX711_LC1.4 (Pin_4)
- new net: J_Encoder_1.3 (Pin_3), R27.2
- new net: J_Encoder_2.4 (Pin_4), R33.2
- new net: J_Encoder_2.3 (Pin_3), R31.2
- new net: J_Encoder_1.4 (Pin_4), R29.2
Other:
- moved on the sheet: J3, J4, J_HX711_LC1, J_MD2, R21, R22, R23, R24, U2

Commit message: final pcb
Parts:
- removed R17, R19, R21, R23: 1.8kΩ, Resistor_THT:R_Axial_DIN0207_L6.3mm_D2.5mm_P7.62mm_Horizontal, symbol Device:R
- R18, R20, R22, R24: value 3.3kΩ -> 3.9kΩ
Connections:
- net GPIO1: now also J_MD1.3 (Pin_4)
- net GPIO2: now also J_MD1.4 (Pin_3)
- net GPIO3: now also J_MD2.3 (Pin_4)
- net GPIO4: now also J_MD2.4 (Pin_3)
