File: SPRO-3-PCB/SPRO-3-PCB.kicad_sch (KiCad schematic)
At the start: 71 parts, among them J1 Screw_Terminal_01x02, J2 Micro_SD_Card, J3 Conn_01x22, J4 Conn_01x22, Q1 IRF4905, U1 TSR_1-2450, U2 ESP32-S3-DEVKITC-1-N8R2, U6 LD1117V33

Commit message: Add files via upload
Connections:
- net GPIO19: no longer R14.2, R15.1
- net GPIO20: no longer J_IR1.1 (Pin_1), R4.1
- net GPIO21: now also J_HX711_LC1.4 (Pin_4), R27.1, R28.2; no longer J_IR2.1 (Pin_1), R5.2
- net GPIO35: no longer J_HX711_LC1.4 (Pin_4)
- net GPIO36: no longer R27.1, R28.2
- net GPIO37: no longer R29.1, R30.1
- net GPIO39: now also J_MD1.7 (Pin_8)
- net GPIO40: now also J_MD1.8 (Pin_7)
- net GPIO41: now also J_MD2.7 (Pin_8)
- net GPIO42: now also J_MD2.8 (Pin_7); no longer J_IR3.1 (Pin_1), R6.2
- net GPIO47: now also R29.1, R30.1
- net GPIO5: now also J_IR1.1 (Pin_1), R4.1; no longer J_MD1.7 (Pin_8)
- net GPIO6: now also J_IR2.1 (Pin_1), R5.2; no longer J_MD1.8 (Pin_7)
- net GPIO7: now also J_IR3.1 (Pin_1), R6.2; no longer J_MD2.7 (Pin_8)
- net GPIO8: now also R14.2, R15.1; no longer J_MD2.8 (Pin_7)

Commit message: Add files via upload
Parts:
- removed R18, R20, R22, R24: 3.9kΩ, Resistor_THT:R_Axial_DIN0207_L6.3mm_D2.5mm_P7.62mm_Horizontal, symbol Device:R
Connections:
- net GPIO1: now also R27.1, R28.2; no longer J_MD1.3 (Pin_4)
- net GPIO14: now also R10.2, R11.1; no longer J_US1.2 (Pin_2)
- net GPIO15: now also R12.2, R13.1; no longer R10.2, R11.1
- net GPIO16: now also R14.2, R15.1; no longer J_US2.2 (Pin_2)
- net GPIO17: now also R31.1, R32.2; no longer R12.2, R13.1
- net GPIO18: now also R33.1, R34.1; no longer J_US3.2 (Pin_2)
- net GPIO2: now also R29.1, R30.1; no longer J_MD1.4 (Pin_3)
- net GPIO21: no longer R27.1, R28.2
- net GPIO3: no longer J_MD2.3 (Pin_4)
- net GPIO38: no longer R31.1, R32.2
- net GPIO39: no longer R33.1, R34.1
- net GPIO4: now also J_US1.2 (Pin_2), J_US2.2 (Pin_2), J_US3.2 (Pin_2); no longer J_MD2.4 (Pin_3)
- net GPIO47: no longer R29.1, R30.1
- net GPIO5: now also J_IR3.1 (Pin_1), R6.2; no longer J_IR1.1 (Pin_1), R4.1
- net GPIO7: now also J_IR1.1 (Pin_1), R4.1; no longer J_IR3.1 (Pin_1), R6.2
- net GPIO8: no longer R14.2, R15.1
- no-connect marks 2 -> 6
Other:
- moved on the sheet: C11, C12, C13, C14, C15, C16, J_Encoder_1, J_Encoder_2, J_MD1, J_MD2, R27, R28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
