File: SPRO-3-PCB/SPRO-3-PCB.kicad_pcb (KiCad board)
At the start: 2 copper layers, 124.2 x 142 mm, 71 parts, among them J1 Screw_Terminal_01x02, J2 Micro_SD_Card, J3 Conn_01x22, J4 Conn_01x22, Q1 IRF4905, U1 TSR_1-2450, U2 ESP32-S3-DEVKITC-1-N8R2, U6 LD1117V33

Commit message: Add files via upload
Parts:
- removed R18, R20, R22, R24: 3.9kΩ, Resistor_THT:R_Axial_DIN0207_L6.3mm_D2.5mm_P7.62mm_Horizontal
Connections:
- J_HX711_LC1 pad 4: GPIO35 -> GPIO21
- J_IR1 pad 1: GPIO20 -> GPIO7
- J_IR2 pad 1: GPIO21 -> GPIO6
- J_IR3 pad 1: GPIO42 -> GPIO5
- J_MD1 pad 3: GPIO1 -> unconnected-(J_MD1-Pin_4-Pad3)
- J_MD1 pad 4: GPIO2 -> unconnected-(J_MD1-Pin_3-Pad4)
- J_MD1 pad 7: GPIO5 -> GPIO39
- J_MD1 pad 8: GPIO6 -> GPIO40
- J_MD2 pad 3: GPIO3 -> unconnected-(J_MD2-Pin_4-Pad3)
- J_MD2 pad 4: GPIO4 -> unconnected-(J_MD2-Pin_3-Pad4)
- J_MD2 pad 7: GPIO7 -> GPIO41
- J_MD2 pad 8: GPIO8 -> GPIO42
- J_US1 pad 2: GPIO14 -> GPIO4
- J_US2 pad 2: GPIO16 -> GPIO4
- J_US3 pad 2: GPIO18 -> GPIO4
- R10 pad 2: GPIO15 -> GPIO14
- R11 pad 1: GPIO15 -> GPIO14
- R12 pad 2: GPIO17 -> GPIO15
- R13 pad 1: GPIO17 -> GPIO15
- R14 pad 2: GPIO19 -> GPIO16
- R15 pad 1: GPIO19 -> GPIO16
- R27 pad 1: GPIO36 -> GPIO1
- R28 pad 2: GPIO36 -> GPIO1
- R29 pad 1: GPIO37 -> GPIO2
- R30 pad 1: GPIO37 -> GPIO2
- R31 pad 1: GPIO38 -> GPIO17
- R32 pad 2: GPIO38 -> GPIO17
- R33 pad 1: GPIO39 -> GPIO18
- R34 pad 1: GPIO39 -> GPIO18
- R4 pad 1: GPIO20 -> GPIO7
- R5 pad 2: GPIO21 -> GPIO6
- R6 pad 2: GPIO42 -> GPIO5
Routing:
- net GPIO38: track 151.8 -> 16.8 mm, vias 1 -> 0
- net GPIO36: track 126.7 -> 16.1 mm, vias 1 -> 0
- net GPIO37: track 126.2 -> 16.1 mm, vias 1 -> 0
- net GPIO41: track 16.1 -> 125.5 mm, vias 0 -> 1
- net GPIO17: track 34.7 -> 122.2 mm, vias 0 -> 1
- net GPIO42: track 41.9 -> 129.2 mm, vias 0 -> 1
- net GPIO35: track 103.2 -> 16.1 mm, vias 3 -> 0
- net GPIO19: track 102.8 -> 16.1 mm
- net GPIO40: track 16.1 -> 102.2 mm
- net GPIO8: track 93.2 -> 16.1 mm, vias 2 -> 0
- net GPIO3: track 92.2 -> 16.1 mm
- net GPIO18: track 47.1 -> 121.8 mm, vias 0 -> 2
- net GPIO39: track 167.3 -> 103.8 mm, vias 1 -> 0
- net GPIO21: track 52.3 -> 107.3 mm, vias 0 -> 2
- net GPIO5: track 99.7 -> 154.2 mm, vias 2 -> 0
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Other:
- outline, holes or cut-outs redrawn

Commit message: final design
Parts:
- moved C7 5.75 mm to (58.8, 38.0)
- moved C15 4.32 mm to (114.1, 25.6)
- moved C16 4.32 mm to (124.6, 25.6)
- moved J_Encoder_1 4.32 mm to (116.7, 29.7)
- moved R27 4.32 mm to (112.1, 41.9)
- moved R28 4.32 mm to (116.1, 49.5)
- moved R29 4.32 mm to (108.6, 41.9)
- moved R30 4.32 mm to (104.6, 41.9)
- moved R31 4.32 mm to (126.6, 41.9)
- moved R32 4.32 mm to (122.8, 49.5)
- moved R33 4.32 mm to (130.3, 41.9)
- moved R34 4.32 mm to (134.3, 41.9)
- moved J_Encoder_2 4.32 mm to (122.1, 29.7)
- moved Q1 4.00 mm to (56.5, 29.0)
- moved R16 3.50 mm to (63.8, 33.1)
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Routing:
- net GND: track 203.6 -> 287.3 mm
- net GPIO17: track 122.2 -> 132.2 mm
- net +5V: track 371.9 -> 363.4 mm
- net +12V: track 103.2 -> 95.8 mm
- net Net-(J_Switch1-Pin_1): track 14.7 -> 10.7 mm
- net GPIO2: track 138.9 -> 141.9 mm
- net GPIO18: track 121.8 -> 120.3 mm
- net GPIO1: track 147.5 -> 148.0 mm, vias 1 -> 2
- net Net-(Q1-G): track 8.44 -> 8.94 mm
Other:
- board size 124.2 x 142 mm -> 124.2 x 144.2 mm
- board text added: "Group 1C"
- board text added: "SPRO-3"
